File: i2c_bus_magslide.kicad_sch (KiCad schematic)
At the start: 16 parts, among them J1 50-00174, J10 50-00174, J11 uC Connector, J12 Debug Connector, J2 50-00174, J3 50-00174, J4 50-00174, J5 50-00174, J6 50-00174, J7 50-00174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

Commit message: Inc
Parts:
- added H1, H2: MountingHole, MountingHole:MountingHole_3.2mm_M3, symbol Mechanical:MountingHole
- J1, J10, J2, J3, J4, J5, J6, J7, J8, J9: footprint (none) -> misc:54-00174
- J11: footprint (none) -> Connector_PinHeader_2.54mm:PinHeader_1x05_P2.54mm_Vertical
- J12: footprint (none) -> Connector_PinHeader_2.54mm:PinHeader_1x03_P2.54mm_Vertical
- JP1, JP2: footprint (none) -> Jumper:SolderJumper-2_P1.3mm_Open_RoundedPad1.0x1.5mm
- R1, R2: footprint (none) -> Resistor_THT:R_Box_L8.4mm_W2.5mm_P5.08mm
